File: RP2040circuitry.kicad_sch (KiCad schematic)
At the start: 0 parts

Commit message: Refactor code structure and remove redundant sections for improved readability and maintainability
Parts:
- added C1, C2: 10u, symbol Device:C
- added J1: TYPE-C-31-M-12, usb-c:HRO_TYPE-C-31-M-12, symbol TYPE-C-31-M-12:TYPE-C-31-M-12
- added R1, R2: 5.1k, symbol Device:R
- added U1: RP2040, RP2040_minimal_r2:RP2040-QFN-56, symbol MCU_RaspberryPi_RP2040:RP2040
- added U2: NCP1117-3.3_SOT223, Package_TO_SOT_SMD:SOT-223-3_TabPin2, symbol Regulator_Linear:NCP1117-3.3_SOT223
Connections:
- new net: J1.A5 (CC1), R2.1
- new net: J1.B5 (CC2), R1.1
- new net +3V3: C2.1, U2.2 (VO)
- new net GND: C1.2, C2.2, J1.A1_B12 (GND), J1.B1_A12 (GND), J1.S1 (SHIELD), J1.S2 (SHIELD), J1.S3 (SHIELD), J1.S4 (SHIELD), R1.2, R2.2, U2.1 (GND)
- new net USB D+: J1.A6 (DP1), J1.B6 (DP2)
- new net USB D-: J1.A7 (DN1), J1.B7 (DN2)
- new net VBUS: C1.1, J1.A4_B9 (VBUS), J1.B4_A9 (VBUS), U2.3 (VI)
- no-connect marks 0 -> 2

Commit message: Added shematic changes!
Parts:
- added C10, C3: 1u, symbol Device:C
- added C11, C12, C13, C14, C4, C5, C6, C7, C8, C9: 100n, symbol Device:C
- added SW1: SW_Push, symbol Switch:SW_Push
- added U3: W25Q128JVS, Package_SO:SOIC-8_5.3x5.3mm_P1.27mm, symbol Memory_Flash:W25Q128JVS
Connections:
- net +3V3: now also U1.1 (IOVDD), U1.10 (IOVDD), U1.22 (IOVDD), U1.33 (IOVDD), U1.42 (IOVDD), U1.43 (ADC_AVDD), U1.44 (VREG_IN), U1.48 (USB_VDD), U1.49 (IOVDD), C11.1, C14.1, C3.1, C4.1, C5.1, C6.1, C7.1, C8.1, C9.1, SW1.2, U3.1 (~{CS}), U3.8 (VCC)
- net GND: now also C10.2, C11.2, C12.2, C13.2, C14.2, C3.2, C4.2, C5.2, C6.2, C7.2, C8.2, C9.2, SW1.1, U3.4 (GND)
- net +1V1: now reaches U1.23 (DVDD)
- net +1V1: now also U1.45 (VREG_VOUT), U1.50 (DVDD), C10.1, C12.1, C13.1
- new net FLASH_0: U3.5 (DI/IO_{0})
- new net FLASH_1: U3.2 (DO/IO_{1})
- new net FLASH_2: U3.3 (~{WP}/IO_{2})
- new net FLASH_3: U3.7 (~{HOLD}/~{RESET}/IO_{3})
- new net FLASH_CLK: U3.6 (CLK)
Other:
- note added: "Close to pin 44"
- note added: "Close to pin 45"
- note added: "Flash + Boot control"
- note added: "USB Port + 3v3 LDO"
- moved on the sheet: C1, C2, J1, R1, R2, U1, U2

Commit message: added crystal osccillator
Parts:
- added C15, C16: C, symbol Device:C
- added R3, R4: 1k, symbol Device:R
- added X1: ABM8-272-T3, ABM8-272-T3_ABR, symbol 2025-01-15_21-49-59:ABM8-272-T3
Connections:
- net +3V3: now also U1.56 (QSPI_SS), R3.2; no longer SW1.2
- net FLASH_0: now also U1.53 (QSPI_SD0)
- net FLASH_1: now also U1.55 (QSPI_SD1)
- net FLASH_2: now also U1.54 (QSPI_SD2)
- net FLASH_3: now also U1.51 (QSPI_SD3)
- net FLASH_CLK: now also U1.52 (QSPI_SCLK)
- net GND: now also C15.1, C16.1, X1.2, X1.4
- new net: C15.2, R4.1, X1.3
- new net: R3.1, SW1.2
- new net XIN: C16.2, X1.1
- new net XOUT: R4.2
Other:
- note added: "Close to flash chip"
- note added: "Crystal Oscillator"
- moved on the sheet: C14, SW1, U3

Commit message: Power + Optocoupler
Parts:
- X1: footprint ABM8-272-T3_ABR -> footprints:ABM8-272-T3_ABR
Connections:
- net XIN: now also U1.20 (XIN)
- net XOUT: now also U1.21 (XOUT)
Changed lines of the file:
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@@
 	(generator "eeschema")
 	(generator_version "9.0")
-	(paper "A4")
+	(paper "A3")
 	(rectangle
 		(start 20.32 154.94)
@@
 	(wire
 		(pts
+			(xy 166.37 111.76) (xy 175.26 111.76)
+		)
+		(stroke
+			(width 0)
+			(type default)
+		)
+	)
+	(wire
+		(pts
 			(xy 213.36 55.88) (xy 215.9 55.88)
 		)
@@
 	(wire
 		(pts
+			(xy 166.37 116.84) (xy 175.26 116.84)
+		)
+		(stroke
+			(width 0)
+			(type default)
+		)
+	)
+	(wire
+		(pts
 			(xy 186.69 55.88) (xy 186.69 58.42)
 		)
@@
 		)
 	)
+	(label "XOUT"
+		(at 166.37 116.84 0)
+		(effects
+			(font
+				(size 1.27 1.27)
+			)
+			(justify left bottom)
+		)
+	)
+	(label "XIN"
+		(at 166.37 111.76 0)
+		(effects
+			(font
+				(size 1.27 1.27)
+			)
+			(justify left bottom)
+		)
+	)
 	(label "XIN"
 		(at 109.22 161.29 180)
@@
 			)
 		)
-		(property "Footprint" "ABM8-272-T3_ABR"
+		(property "Footprint" "footprints:ABM8-272-T3_ABR"
 			(at 53.34 171.45 0)
 			(effects

Commit message: BOM + footprints
Parts:
- added R7, R8: 27, symbol Device:R
- C15, C16: value C -> 15p
Connections:
- net USB D+: now also R8.2
- net USB D-: now also R7.2
- net at U1.46 (USB_DM): now also R8.1
- net at U1.47 (USB_DP): now also R7.1
Changed lines of the file:
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@@
 	(wire
 		(pts
+			(xy 257.81 58.42) (xy 267.97 58.42)
+		)
+		(stroke
+			(width 0)
+			(type default)
+		)
+	)
+	(wire
+		(pts
 			(xy 44.45 109.22) (xy 53.34 109.22)
 		)
@@
 	(wire
 		(pts
+			(xy 257.81 68.58) (xy 267.97 68.58)
+		)
+		(stroke
+			(width 0)
+			(type default)
+		)
+	)
+	(wire
+		(pts
 			(xy 270.51 38.1) (xy 280.67 38.1)
 		)
@@
 	(wire
 		(pts
+			(xy 238.76 68.58) (xy 250.19 68.58)
+		)
+		(stroke
+			(width 0)
+			(type default)
+		)
+	)
+	(wire
+		(pts
 			(xy 78.74 182.88) (xy 49.53 182.88)
 		)
@@
 	(wire
 		(pts
+			(xy 245.11 58.42) (xy 245.11 66.04)
+		)
+		(stroke
+			(width 0)
+			(type default)
+		)
+	)
+	(wire
+		(pts
 			(xy 41.91 171.45) (xy 41.91 182.88)
 		)
@@
 	(wire
 		(pts
+			(xy 250.19 58.42) (xy 245.11 58.42)
+		)
+		(stroke
+			(width 0)
+			(type default)
+		)
+	)
+	(wire
+		(pts
 			(xy 250.19 38.1) (xy 260.35 38.1)
 		)
@@
 	(wire
 		(pts
+			(xy 245.11 66.04) (xy 238.76 66.04)
+		)
+		(stroke
+			(width 0)
+			(type default)
+		)
+	)
+	(wire
+		(pts
 			(xy 161.29 88.9) (xy 175.26 88.9)
 		)
@@
 		)
 	)
+	(global_label "USB D+"
+		(shape input)
+		(at 267.97 68.58 0)
+		(fields_autoplaced yes)
+		(effects
+			(font
+				(size 1.27 1.27)
+			)
+			(justify left)
+		)
+		(property "Intersheetrefs" "${INTERSHEET_REFS}"
+			(at 278.5752 68.58 0)
+			(effects
+				(font
+					(size 1.27 1.27)
+				)
+				(justify left)
+				(hide yes)
+			)
+		)
+	)
+	(global_label "USB D-"
+		(shape input)
+		(at 267.97 58.42 0)
+		(fields_autoplaced yes)
+		(effects
+			(font
+				(size 1.27 1.27)
+			)
+			(justify left)
+		)
+		(property "Intersheetrefs" "${INTERSHEET_REFS}"
+			(at 278.5752 58.42 0)
+			(effects
+				(font
+					(size 1.27 1.27)
+				)
+				(justify left)
+				(hide yes)
+			)
+		)
+	)
 	(global_label "USB D-"
 		(shape input)
@@
 			)
 		)
-		(property "Value" "C"
+		(property "Value" "15p"
 			(at 45.72 177.8 90)
 			(effects
@@
 	(symbol
 		(lib_id "Device:R")
+		(at 254 68.58 90)
+		(unit 1)
+		(exclude_from_sim no)
+		(in_bom yes)
+		(on_board yes)
+		(dnp no)
+		(fields_autoplaced yes)
+		(property "Reference" "R8"
+			(at 254 62.23 90)
+			(effects
+				(font
+					(size 1.27 1.27)
+				)
+			)
+		)
+		(property "Value" "27"
+			(at 254 64.77 90)
+			(effects
+				(font
+					(size 1.27 1.27)
+				)
+			)
+		)
+		(property "Footprint" ""
+			(at 254 70.358 90)
+			(effects
+				(font
+					(size 1.27 1.27)
+				)
+				(hide yes)
+			)
+		)
+		(property "Datasheet" "~"
+			(at 254 68.58 0)
+			(effects
+				(font
+					(size 1.27 1.27)
+				)
+				(hide yes)
+			)
+		)
+		(property "Description" "Resistor"
+			(at 254 68.58 0)
+			(effects
+				(font
+					(size 1.27 1.27)
+				)
+				(hide yes)
+			)
+		)
+		(pin "2"
+		)
+		(pin "1"
+		)
+		(instances
+			(project "NeoPWM"
+				(path "/5f4f8df1-f390-4405-b7ce-064ebaa7e775/883e8582-d657-46a8-8863-9bdb5189a894"
+					(reference "R8")
+					(unit 1)
+				)
+			)
+		)
+	)
+	(symbol
+		(lib_id "Device:R")
 		(at 40.64 109.22 90)
 		(unit 1)
@@
 		(on_board yes)
 		(dnp no)
-		(fields_autoplaced yes)
 		(property "Reference" "SW1"
 			(at 29.21 113.0299 90)
@@
 			)
 		)
-		(property "Value" "C"
+		(property "Value" "15p"
 			(at 45.72 166.37 90)
 			(effects
@@
 					(unit 1)
 				)
+			)
+		)
+	)
+	(symbol
+		(lib_id "Device:R")
+		(at 254 58.42 90)
+		(unit 1)
+		(exclude_from_sim no)
+		(in_bom yes)
+		(on_board yes)
+		(dnp no)
+		(property "Reference" "R7"
+			(at 254 52.07 90)
+			(effects
+				(font
+					(size 1.27 1.27)
+				)
+			)
+		)
+		(property "Value" "27"
+			(at 254 54.61 90)
+			(effects
+				(font
+					(size 1.27 1.27)
+				)
+			)
+		)
+		(property "Footprint" ""
+			(at 254 60.198 90)
+			(effects
+				(font
+					(size 1.27 1.27)
+				)
+				(hide yes)
+			)
+		)
+		(property "Datasheet" "~"
+			(at 254 58.42 0)
+			(effects
+				(font
+					(size 1.27 1.27)
+				)
+				(hide yes)
+			)
+		)
+		(property "Description" "Resistor"
+			(at 254 58.42 0)
+			(effects
+				(font
+					(size 1.27 1.27)
+				)
+				(hide yes)
+			)
+		)
+		(pin "2"
+		)
+		(pin "1"
+		)
+		(instances
+			(project ""
+				(path "/5f4f8df1-f390-4405-b7ce-064ebaa7e775/883e8582-d657-46a8-8863-9bdb5189a894"
+					(reference "R7")
+					(unit 1)
+				)

Commit message: 3D Models
Parts:
- C1, C10, C11, C12, C13, C14, C15, C16, C2, C3, C4, C5, C6, C7, C8, C9: footprint (none) -> Capacitor_SMD:C_0402_1005Metric
- R1, R2, R3, R4, R7, R8: footprint (none) -> Resistor_SMD:R_0402_1005Metric
- SW1: footprint (none) -> TS-1088-AR02016:SW_TS-1088_XNP-L
Changed lines of the file:
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@@
 	(wire
 		(pts
+			(xy 289.56 64.77) (xy 306.07 64.77)
+		)
+		(stroke
+			(width 0)
+			(type default)
+		)
+	)
+	(wire
+		(pts
 			(xy 100.33 107.95) (xy 100.33 110.49)
 		)
@@
 	(wire
 		(pts
+			(xy 289.56 71.12) (xy 306.07 71.12)
+		)
+		(stroke
+			(width 0)
+			(type default)
+		)
+	)
+	(wire
+		(pts
 			(xy 238.76 68.58) (xy 250.19 68.58)
 		)
@@
 		)
 	)
+	(label "NeoPixel 5v"
+		(at 306.07 64.77 180)
+		(effects
+			(font
+				(size 1.27 1.27)
+			)
+			(justify right bottom)
+		)
+	)
 	(label "FLASH_1"
 		(at 59.69 116.84 0)
@@
 		)
 	)
+	(label "NeoPixel Signal"
+		(at 293.37 81.28 0)
+		(effects
+			(font
+				(size 1.27 1.27)
+			)
+			(justify left bottom)
+		)
+	)
 	(label "FLASH_2"
 		(at 59.69 119.38 0)
@@
 		)
 	)
+	(label "NeoPixel GND"
+		(at 306.07 71.12 180)
+		(effects
+			(font
+				(size 1.27 1.27)
+			)
+			(justify right bottom)
+		)
+	)
 	(label "FLASH_SS"
 		(at 161.29 77.47 0)
@@
 			)
 		)
-		(property "Footprint" ""
+		(property "Footprint" "Capacitor_SMD:C_0402_1005Metric"
 			(at 261.3152 38.1 0)
 			(effects
@@
 			)
 		)
-		(property "Footprint" ""
+		(property "Footprint" "Capacitor_SMD:C_0402_1005Metric"
 			(at 167.3352 36.83 0)
 			(effects
@@
 	(symbol
 		(lib_id "power:GND")
+		(at 289.56 71.12 0)
+		(unit 1)
+		(exclude_from_sim no)
+		(in_bom yes)
+		(on_board yes)
+		(dnp no)
+		(fields_autoplaced yes)
+		(property "Reference" "#PWR025"
+			(at 289.56 77.47 0)
+			(effects
+				(font
+					(size 1.27 1.27)
+				)
+				(hide yes)
+			)
+		)
+		(property "Value" "GND"
+			(at 289.56 76.2 0)
+			(effects
+				(font
+					(size 1.27 1.27)
+				)
+			)
+		)
+		(property "Footprint" ""
+			(at 289.56 71.12 0)
+			(effects
+				(font
+					(size 1.27 1.27)
+				)
+				(hide yes)
+			)
+		)
+		(property "Datasheet" ""
+			(at 289.56 71.12 0)
+			(effects
+				(font
+					(size 1.27 1.27)
+				)
+				(hide yes)
+			)
+		)
+		(property "Description" "Power symbol creates a global label with name \"GND\" , ground"
+			(at 289.56 71.12 0)
+			(effects
+				(font
+					(size 1.27 1.27)
+				)
+				(hide yes)
+			)
+		)
+		(pin "1"
+		)
+		(instances
+			(project ""
+				(path "/5f4f8df1-f390-4405-b7ce-064ebaa7e775/883e8582-d657-46a8-8863-9bdb5189a894"
+					(reference "#PWR025")
+					(unit 1)
+				)
+			)
+		)
+	)
+	(symbol
+		(lib_id "power:GND")
 		(at 100.33 110.49 0)
 		(unit 1)
@@
 			)
 		)
-		(property "Footprint" ""
+		(property "Footprint" "Capacitor_SMD:C_0402_1005Metric"
 			(at 281.6352 38.1 0)
 			(effects
@@
 			)
 		)
-		(property "Footprint" ""
+		(property "Footprint" "Capacitor_SMD:C_0402_1005Metric"
 			(at 49.53 181.9148 0)
 			(effects
@@
 			)
 		)
-		(property "Footprint" ""
+		(property "Footprint" "Capacitor_SMD:C_0402_1005Metric"
 			(at 140.6652 50.8 0)
 			(effects
@@
 			)
 		)
-		(property "Footprint" ""
+		(property "Footprint" "Capacitor_SMD:C_0402_1005Metric"
 			(at 271.4752 38.1 0)
 			(effects
@@
 			)
 		)
-		(property "Footprint" ""
+		(property "Footprint" "Resistor_SMD:R_0402_1005Metric"
 			(at 254 70.358 90)
 			(effects
@@
 			)
 		)
-		(property "Footprint" ""
+		(property "Footprint" "Resistor_SMD:R_0402_1005Metric"
 			(at 40.64 110.998 90)
 			(effects
@@
 			)
 		)
-		(property "Footprint" ""
+		(property "Footprint" "Capacitor_SMD:C_0402_1005Metric"
 			(at 291.7952 38.1 0)
 			(effects
@@
 			)
 		)
-		(property "Footprint" ""
+		(property "Footprint" "Capacitor_SMD:C_0402_1005Metric"
 			(at 101.2952 107.95 0)
 			(effects
@@
 			)
 		)
-		(property "Footprint" ""
+		(property "Footprint" "TS-1088-AR02016:SW_TS-1088_XNP-L"
 			(at 22.86 114.3 0)
 			(effects
@@
 			)
 		)
-		(property "Footprint" ""
+		(property "Footprint" "Capacitor_SMD:C_0402_1005Metric"
 			(at 251.1552 38.1 0)
 			(effects
@@
 			)
 		)
-		(property "Footprint" ""
+		(property "Footprint" "Capacitor_SMD:C_0402_1005Metric"
 			(at 112.7252 50.8 0)
 			(effects
@@
 			)
 		)
-		(property "Footprint" ""
+		(property "Footprint" "Resistor_SMD:R_0402_1005Metric"
 			(at 28.702 52.07 90)
 			(effects
@@
 			)
 		)
-		(property "Footprint" ""
+		(property "Footprint" "Resistor_SMD:R_0402_1005Metric"
 			(at 92.71 175.768 90)
 			(effects
@@
 			)
 		)
-		(property "Footprint" ""
+		(property "Footprint" "Capacitor_SMD:C_0402_1005Metric"
 			(at 230.8352 38.1 0)
 			(effects
@@
 			)
 		)
-		(property "Footprint" ""
+		(property "Footprint" "Capacitor_SMD:C_0402_1005Metric"
 			(at 240.9952 38.1 0)
 			(effects
@@
 			)
 		)
-		(property "Footprint" ""
+		(property "Footprint" "Capacitor_SMD:C_0402_1005Metric"
 			(at 49.53 170.4848 0)
 			(effects
@@
 			)
 		)
-		(property "Footprint" ""
+		(property "Footprint" "Resistor_SMD:R_0402_1005Metric"
 			(at 87.122 58.42 90)
 			(effects
@@
 	(symbol
 		(lib_id "power:VBUS")
+		(at 289.56 64.77 0)
+		(unit 1)
+		(exclude_from_sim no)
+		(in_bom yes)
+		(on_board yes)
+		(dnp no)
+		(fields_autoplaced yes)
+		(property "Reference" "#PWR024"
+			(at 289.56 68.58 0)
+			(effects
+				(font
+					(size 1.27 1.27)
+				)
+				(hide yes)
+			)
+		)
+		(property "Value" "VBUS"
+			(at 289.56 59.69 0)
+			(effects
+				(font
+					(size 1.27 1.27)
+				)
+			)
+		)
+		(property "Footprint" ""
+			(at 289.56 64.77 0)
+			(effects
+				(font
+					(size 1.27 1.27)
+				)
+				(hide yes)
+			)
+		)
+		(property "Datasheet" ""
+			(at 289.56 64.77 0)
+			(effects
+				(font
+					(size 1.27 1.27)
+				)
+				(hide yes)
+			)
+		)
+		(property "Description" "Power symbol creates a global label with name \"VBUS\""
+			(at 289.56 64.77 0)
+			(effects
+				(font
+					(size 1.27 1.27)
+				)
+				(hide yes)
+			)
+		)
+		(pin "1"
+		)
+		(instances
+			(project ""
+				(path "/5f4f8df1-f390-4405-b7ce-064ebaa7e775/883e8582-d657-46a8-8863-9bdb5189a894"
+					(reference "#PWR024")
+					(unit 1)
+				)
+			)
+		)
+	)
+	(symbol
+		(lib_id "power:VBUS")
 		(at 97.79 40.64 0)
 		(unit 1)
@@
 			)
 		)
-		(property "Footprint" ""
+		(property "Footprint" "Capacitor_SMD:C_0402_1005Metric"
 			(at 229.5652 52.07 0)
 			(effects
@@
 			)
 		)
-		(property "Footprint" ""
+		(property "Footprint" "Capacitor_SMD:C_0402_1005Metric"
 			(at 177.4952 52.07 0)
 			(effects
@@
 			)
 		)
-		(property "Footprint" ""
+		(property "Footprint" "Capacitor_SMD:C_0402_1005Metric"
 			(at 177.4952 36.83 0)
 			(effects
@@
 			)
 		)
-		(property "Footprint" ""
+		(property "Footprint" "Resistor_SMD:R_0402_1005Metric"
 			(at 254 60.198 90)
 			(effects

Commit message: ahaha
Parts:
- added R9: 10k, Resistor_SMD:R_0402_1005Metric, symbol Device:R
Connections:
- net +3V3: now also R9.1; no longer R3.2, U1.56 (QSPI_SS), U3.1 (~{CS})
- net GND: now also U1.57 (GND)
- net NeoPixel Signal: now also U1.2 (GPIO0)
- net ADC3: now reaches J1.A5 (CC1), R2.1
- net ADC3: now also U1.41 (GPIO29_ADC3)
- net PWM Signal GPIO: now reaches U1.37 (GPIO25)
- net ADC2: now reaches U1.40 (GPIO28_ADC2)
- net ADC2: now also J1.B5 (CC2), R1.1
- new net FLASH_SS: R3.2, R9.2, U1.56 (QSPI_SS), U3.1 (~{CS})
