File: NeoPWM.kicad_pcb (KiCad board)
At the start: 2 copper layers, 2 parts, among them J1 TYPE-C-31-M-12, U1 RP2040

Commit message: Finished schematic
Parts:
- added C1: 10u, Capacitor_SMD:C_0402_1005Metric, F.Cu at (44.7, 30.8)
- added C10: 1u, Capacitor_SMD:C_0402_1005Metric, F.Cu at (50.5, 32.8)
- added C11: 100n, Capacitor_SMD:C_0402_1005Metric, F.Cu at (50.5, 34.7)
- added C12: 100n, Capacitor_SMD:C_0402_1005Metric, F.Cu at (50.5, 36.7)
- added C13: 100n, Capacitor_SMD:C_0402_1005Metric, F.Cu at (53.3, 30.8)
- added C14: 100n, Capacitor_SMD:C_0402_1005Metric, F.Cu at (53.3, 32.8)
- added C15: 15p, Capacitor_SMD:C_0402_1005Metric, F.Cu at (53.3, 34.7)
- added C16: 15p, Capacitor_SMD:C_0402_1005Metric, F.Cu at (53.3, 36.7)
- added C2: 10u, Capacitor_SMD:C_0402_1005Metric, F.Cu at (44.7, 32.8)
- added C3: 1u, Capacitor_SMD:C_0402_1005Metric, F.Cu at (44.7, 34.7)
- added C4: 100n, Capacitor_SMD:C_0402_1005Metric, F.Cu at (44.7, 36.7)
- added C5: 100n, Capacitor_SMD:C_0402_1005Metric, F.Cu at (47.6, 30.8)
- added C6: 100n, Capacitor_SMD:C_0402_1005Metric, F.Cu at (47.6, 32.8)
- added C7: 100n, Capacitor_SMD:C_0402_1005Metric, F.Cu at (47.6, 34.7)
- added C8: 100n, Capacitor_SMD:C_0402_1005Metric, F.Cu at (47.6, 36.7)
- added C9: 100n, Capacitor_SMD:C_0402_1005Metric, F.Cu at (50.5, 30.8)
- added J2: PWM Input, Connector_PinHeader_2.54mm:PinHeader_1x03_P2.54mm_Horizontal, F.Cu at (53.4, 59.4)
- added J3: NeoPixel Connector, 691137710003:CONN3_WR-TBL-1377_WRE, F.Cu at (44.8, 51.4)
- added R1: 5.1k, Resistor_SMD:R_0402_1005Metric, F.Cu at (41.8, 30.8)
- added R2: 5.1k, Resistor_SMD:R_0402_1005Metric, F.Cu at (41.8, 32.8)
- added R3: 1k, Resistor_SMD:R_0402_1005Metric, F.Cu at (41.8, 34.8)
- added R4: 1k, Resistor_SMD:R_0402_1005Metric, F.Cu at (41.8, 36.8)
- added R5: 470, Resistor_SMD:R_0402_1005Metric, F.Cu at (41.8, 63.4)
- added R6: 4.7k, Resistor_SMD:R_0402_1005Metric, F.Cu at (41.8, 65.4)
- added R7: 27, Resistor_SMD:R_0402_1005Metric, F.Cu at (41.8, 38.8)
- added R8: 27, Resistor_SMD:R_0402_1005Metric, F.Cu at (41.8, 40.7)
- added SW1: SW_Push, TS-1088-AR02016:SW_TS-1088_XNP-L, F.Cu at (58.2, 40.3)
- added U2: NCP1117-3.3_SOT223, Package_TO_SOT_SMD:SOT-223-3_TabPin2, F.Cu at (59.7, 34.0)
- added U3: W25Q128JVS, Package_SO:SOIC-8_5.3x5.3mm_P1.27mm, F.Cu at (48.5, 41.1)
- added U4: LTV-357T, Package_DIP:DIP-4_W7.62mm, F.Cu at (42.0, 57.8)
- added X1: ABM8-272-T3, footprints:ABM8-272-T3_ABR, F.Cu at (65.4, 41.0)
- moved U1 47.4 mm to (60.6, 24.4)
- moved J1 34.6 mm to (46.4, 26.4)
Connections:
- net Net-(J1-VBUS-PadA4_B9) renamed VBUS
- J1 pad A1_B12: Net-(J1-GND-PadA1_B12) -> GND
- J1 pad A5: unconnected-(J1-CC1-PadA5) -> Net-(J1-CC1)
- J1 pad A6: unconnected-(J1-DP1-PadA6) -> USB D+
- J1 pad A7: unconnected-(J1-DN1-PadA7) -> USB D-
- J1 pad B1_A12: Net-(J1-GND-PadA1_B12) -> GND
- J1 pad B5: unconnected-(J1-CC2-PadB5) -> Net-(J1-CC2)
- J1 pad B6: unconnected-(J1-DP2-PadB6) -> USB D+
- J1 pad B7: unconnected-(J1-DN2-PadB7) -> USB D-
- J1 pad S1: Net-(J1-SHIELD-PadS1) -> GND
- J1 pad S2: Net-(J1-SHIELD-PadS1) -> GND
- J1 pad S3: Net-(J1-SHIELD-PadS1) -> GND
- J1 pad S4: Net-(J1-SHIELD-PadS1) -> GND
- U1 pad 1: unconnected-(U1-IOVDD-Pad1) -> +3V3
- U1 pad 10: unconnected-(U1-IOVDD-Pad10) -> +3V3
- U1 pad 20: unconnected-(U1-XIN-Pad20) -> /RP2040 Circuitry/XIN
- U1 pad 21: unconnected-(U1-XOUT-Pad21) -> /RP2040 Circuitry/XOUT
- U1 pad 22: unconnected-(U1-IOVDD-Pad22) -> +3V3
- U1 pad 23: unconnected-(U1-DVDD-Pad23) -> +1V1
- U1 pad 33: unconnected-(U1-IOVDD-Pad33) -> +3V3
- U1 pad 42: unconnected-(U1-IOVDD-Pad42) -> +3V3
- U1 pad 43: unconnected-(U1-ADC_AVDD-Pad43) -> +3V3
- U1 pad 44: unconnected-(U1-VREG_IN-Pad44) -> +3V3
- U1 pad 45: unconnected-(U1-VREG_VOUT-Pad45) -> +1V1
- U1 pad 46: unconnected-(U1-USB_DM-Pad46) -> Net-(U1-USB_DM)
- U1 pad 47: unconnected-(U1-USB_DP-Pad47) -> Net-(U1-USB_DP)
- U1 pad 48: unconnected-(U1-USB_VDD-Pad48) -> +3V3
- U1 pad 49: unconnected-(U1-IOVDD-Pad49) -> +3V3
- U1 pad 50: unconnected-(U1-DVDD-Pad50) -> +1V1
- U1 pad 51: unconnected-(U1-QSPI_SD3-Pad51) -> /RP2040 Circuitry/FLASH_3
- U1 pad 52: unconnected-(U1-QSPI_SCLK-Pad52) -> /RP2040 Circuitry/FLASH_CLK
- U1 pad 53: unconnected-(U1-QSPI_SD0-Pad53) -> /RP2040 Circuitry/FLASH_0
- U1 pad 54: unconnected-(U1-QSPI_SD2-Pad54) -> /RP2040 Circuitry/FLASH_2
- U1 pad 55: unconnected-(U1-QSPI_SD1-Pad55) -> /RP2040 Circuitry/FLASH_1
- U1 pad 56: unconnected-(U1-QSPI_SS-Pad56) -> +3V3

Commit message: ahaha
Parts:
- added H1: MountingHole_Pad, MountingHole:MountingHole_2.2mm_M2_Pad, F.Cu at (136.6, 81.3)
- added H2: MountingHole_Pad, MountingHole:MountingHole_2.2mm_M2_Pad, F.Cu at (136.6, 87.2)
- added H3: MountingHole_Pad, MountingHole:MountingHole_2.2mm_M2_Pad, F.Cu at (83.0, 108.3)
- added H4: MountingHole_Pad, MountingHole:MountingHole_2.2mm_M2_Pad, F.Cu at (121.8, 108.3)
- added R9: 10k, Resistor_SMD:R_0402_1005Metric, F.Cu at (90.7, 83.0)
- U4: footprint Package_DIP:DIP-4_W7.62mm -> LTV-217-B-G:SOIC127P700X210-4N
- moved C5 91.3 mm to (99.9, 105.6), turned to -90 degrees
- moved R4 89.5 mm to (99.0, 105.7), turned to 90 degrees
- moved C13 88.6 mm to (100.8, 105.6), turned to -90 degrees
- moved C2 88.3 mm to (109.5, 92.8), turned to -90 degrees
- moved C15 87.3 mm to (98.8, 109.3), turned to 90 degrees
- moved C8 86.7 mm to (105.8, 101.0)
- moved C6 86.2 mm to (107.1, 95.2)
- moved C7 85.8 mm to (107.1, 96.6)
- moved U1 85.3 mm to (100.0, 100.0)
- moved C3 83.6 mm to (103.7, 94.0), turned to 90 degrees
- moved C16 81.8 mm to (97.0, 105.9)
- moved C1 81.0 mm to (105.2, 84.6), turned to -90 degrees
- moved R7 80.8 mm to (100.8, 94.0), turned to 90 degrees
- moved C10 80.5 mm to (102.8, 94.0), turned to 90 degrees
- moved R8 80.2 mm to (101.8, 94.0), turned to 90 degrees
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Connections:
- J1 pad A5: Net-(J1-CC1) -> /RP2040 Circuitry/ADC3
- J1 pad B5: Net-(J1-CC2) -> /RP2040 Circuitry/ADC2
- J3 pad 1: /NeoPixel Signal -> VBUS
- J3 pad 2: /NeoPixel 5v -> NeoPixel Signal
- J3 pad 3: /NeoPixel GND -> GND
- R1 pad 1: Net-(J1-CC2) -> /RP2040 Circuitry/ADC2
- R2 pad 1: Net-(J1-CC1) -> /RP2040 Circuitry/ADC3
- R3 pad 2: +3V3 -> /RP2040 Circuitry/FLASH_SS
- U1 pad 2: unconnected-(U1-GPIO0-Pad2) -> NeoPixel Signal
- U1 pad 37: unconnected-(U1-GPIO25-Pad37) -> PWM Signal GPIO
- U1 pad 40: unconnected-(U1-GPIO28_ADC2-Pad40) -> /RP2040 Circuitry/ADC2
- U1 pad 41: unconnected-(U1-GPIO29_ADC3-Pad41) -> /RP2040 Circuitry/ADC3
- U1 pad 56: +3V3 -> /RP2040 Circuitry/FLASH_SS
- U1 pad 57: unconnected-(U1-GND-Pad57) -> GND
- U3 pad 1: +3V3 -> /RP2040 Circuitry/FLASH_SS
Routing:
- net GND: track 0.00 -> 35.1 mm, vias 0 -> 15
- net VBUS: track 0.00 -> 35.0 mm
- net PWM Signal GPIO: track 0.00 -> 29.5 mm, vias 0 -> 2
- net NeoPixel Signal: track 0.00 -> 28.0 mm, vias 0 -> 1
- net /RP2040 Circuitry/ADC2: track 0.00 -> 27.1 mm, vias 0 -> 2
- net /RP2040 Circuitry/ADC3: track 0.00 -> 23.6 mm, vias 0 -> 2
- net /RP2040 Circuitry/FLASH_SS: track 0.00 -> 23.5 mm
- net +1V1: track 0.00 -> 22.3 mm, vias 0 -> 3
- net USB D+: track 0.00 -> 21.5 mm, vias 0 -> 2
- net USB D-: track 0.00 -> 21.5 mm, vias 0 -> 2
- net +3V3: track 0.00 -> 19.9 mm
- net /RP2040 Circuitry/FLASH_1: track 0.00 -> 15.9 mm
- net /RP2040 Circuitry/FLASH_2: track 0.00 -> 12.8 mm
- net /RP2040 Circuitry/FLASH_3: track 0.00 -> 11.5 mm
- net /RP2040 Circuitry/FLASH_CLK: track 0.00 -> 10.4 mm
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- added copper zone on F.Cu, net +1V1
- added copper zone on F.Cu, net +3V3
- added copper zone on F.Cu, net /PWM GND
- added copper zone on B.Cu, net GND
Other:
- board outline added: 43.8 x 40.5 mm

Commit message: stuff
Parts:
- moved H2 53.6 mm to (83.0, 84.5)
- moved H1 15.2 mm to (121.8, 84.4)
- moved C16 6.47 mm to (90.5, 105.2)
- moved X1 5.17 mm to (93.8, 104.4)
- moved R4 4.97 mm to (94.2, 107.3), turned to 0 degrees
- moved C15 4.84 mm to (96.3, 105.0)
Routing:
- net Net-(C15-Pad2): track 4.71 -> 14.2 mm
- net GND: track 35.1 -> 44.1 mm, vias 15 -> 14
- net /RP2040 Circuitry/XOUT: track 2.05 -> 7.07 mm
- net /RP2040 Circuitry/XIN: track 8.79 -> 10.2 mm
- added copper zone on B.Cu, net /PWM GND

Commit message: he
Parts:
- J3: footprint 691137710003:CONN3_WR-TBL-1377_WRE -> Connector_JST:JST_PH_S3B-PH-K_1x03_P2.00mm_Horizontal
- moved R6 16.5 mm to (115.5, 91.6)
- moved U4 13.8 mm to (114.9, 86.4), turned to -90 degrees
- moved H1 11.8 mm to (118.9, 73.0)
- moved H2 11.5 mm to (83.2, 73.0)
- moved J3 9.20 mm to (92.3, 76.3), turned to 180 degrees
- moved R5 8.41 mm to (117.5, 83.2)
- moved J2 7.85 mm to (109.6, 80.1)
- moved H4 2.91 mm to (118.9, 108.1)
- moved H3 0.28 mm to (83.2, 108.1)
- moved U2 0.23 mm to (109.3, 86.6)
Routing:
- net PWM Signal GPIO: track 29.5 -> 17.0 mm, vias 2 -> 1
- net VBUS: track 35.0 -> 26.0 mm
- net GND: track 44.1 -> 53.0 mm, vias 14 -> 13
- net /PWM Signal: track 9.58 -> 5.24 mm
- net NeoPixel Signal: track 28.0 -> 24.7 mm
- net +3V3: track 19.9 -> 22.1 mm
- net Net-(R5-Pad2): track 2.09 -> 1.55 mm
Other:
- board size 43.8 x 40.5 mm -> 41 x 40.5 mm
- board text added: "NeoPWM"
- board text added: "USBC Cable Keepout"
- board text added: "github.com/pythonatsea/neopwm"

Commit message: stuff
Parts:
- moved U4 24.1 mm to (104.7, 108.3), turned to 180 degrees
- moved R5 24.0 mm to (106.6, 104.7)
- moved R6 22.8 mm to (99.5, 107.9), turned to 0 degrees
- moved J2 17.3 mm to (107.5, 97.3), turned to 0 degrees
- moved J3 16.9 mm to (93.7, 93.1), turned to -90 degrees
- moved H2 6.35 mm to (89.6, 73.0)
- moved H3 6.35 mm to (89.6, 108.1)
- moved H1 3.50 mm to (115.4, 73.0)
- moved H4 3.50 mm to (115.4, 108.1)
- moved R3 2.83 mm to (90.8, 82.0)
- moved C11 2.68 mm to (93.8, 100.1)
- moved C7 2.53 mm to (107.1, 94.0)
- moved C2 2.47 mm to (107.1, 92.2), turned to 0 degrees
- moved C6 2.08 mm to (107.1, 93.1)
- moved SW1 1.06 mm to (94.7, 82.0)
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Routing:
- net NeoPixel Signal: track 24.7 -> 4.24 mm, vias 1 -> 0
- net GND: track 53.0 -> 38.9 mm
- net /PWM GND: track 0.00 -> 11.2 mm
- net VBUS: track 26.0 -> 35.6 mm, vias 0 -> 1
- net Net-(C15-Pad2): track 14.2 -> 7.65 mm, vias 0 -> 2
- net Net-(R5-Pad2): track 1.55 -> 5.43 mm
- net PWM Signal GPIO: track 17.0 -> 13.3 mm, vias 1 -> 0
- net /PWM Signal: track 5.24 -> 2.40 mm
- net /RP2040 Circuitry/FLASH_SS: track 23.5 -> 21.1 mm
- net +3V3: track 22.1 -> 20.2 mm
- net Net-(R3-Pad1): track 2.30 -> 1.22 mm
- net USB D-: track 21.5 -> 22.1 mm
- net USB D+: track 21.5 -> 22.1 mm
- net /RP2040 Circuitry/FLASH_1: track 15.9 -> 16.4 mm
- removed copper zone on B.Cu, net /PWM GND
- removed copper zone on F.Cu, net /PWM GND
Other:
- board size 41 x 40.5 mm -> 31.2 x 40.5 mm
