File: Hardware/v0/NeoPWM.kicad_pcb (KiCad board)
At the start: 2 copper layers, 31.2 x 40.5 mm, 38 parts, among them J1 TYPE-C-31-M-12, J2 PWM Input, J3 NeoPixel Connector, SW1 SW_Push, U1 RP2040, U2 NCP1117-3.3_SOT223, U3 W25Q128JVS, U4 LTV-357T, X1 ABM8-272-T3

Commit message: he
Parts:
- added C17: 0.1u, Capacitor_SMD:C_0402_1005Metric, F.Cu at (143.9, 83.5)
- added C18: 0.1u, Capacitor_SMD:C_0402_1005Metric, F.Cu at (143.9, 90.5)
- added C19: 0.1u, Capacitor_SMD:C_0402_1005Metric, F.Cu at (143.9, 97.5)
- added C20: 0.1u, Capacitor_SMD:C_0402_1005Metric, F.Cu at (143.9, 104.5)
- added C21: 0.1u, Capacitor_SMD:C_0402_1005Metric, F.Cu at (151.9, 83.5)
- added C22: 0.1u, Capacitor_SMD:C_0402_1005Metric, F.Cu at (151.9, 90.5)
- added C23: 0.1u, Capacitor_SMD:C_0402_1005Metric, F.Cu at (151.9, 97.5)
- added C24: 0.1u, Capacitor_SMD:C_0402_1005Metric, F.Cu at (151.9, 104.5)
- added C25: 0.1u, Capacitor_SMD:C_0402_1005Metric, F.Cu at (159.9, 83.5)
- added C26: 0.1u, Capacitor_SMD:C_0402_1005Metric, F.Cu at (159.9, 90.5)
- added C27: 0.1u, Capacitor_SMD:C_0402_1005Metric, F.Cu at (159.9, 97.5)
- added C28: 0.1u, Capacitor_SMD:C_0402_1005Metric, F.Cu at (159.9, 104.5)
- added C29: 100u, Capacitor_SMD:C_0402_1005Metric, F.Cu at (139.0, 76.8)
- added D1: SK6812, LED_SMD:LED_SK6812_PLCC4_5.0x5.0mm_P3.2mm, F.Cu at (141.9, 80.0)
- added D10: SK6812, LED_SMD:LED_SK6812_PLCC4_5.0x5.0mm_P3.2mm, F.Cu at (157.9, 87.0)
- added D11: SK6812, LED_SMD:LED_SK6812_PLCC4_5.0x5.0mm_P3.2mm, F.Cu at (157.9, 94.0)
- added D12: SK6812, LED_SMD:LED_SK6812_PLCC4_5.0x5.0mm_P3.2mm, F.Cu at (157.9, 101.0)
- added D2: SK6812, LED_SMD:LED_SK6812_PLCC4_5.0x5.0mm_P3.2mm, F.Cu at (141.9, 87.0)
- added D3: SK6812, LED_SMD:LED_SK6812_PLCC4_5.0x5.0mm_P3.2mm, F.Cu at (141.9, 94.0)
- added D4: SK6812, LED_SMD:LED_SK6812_PLCC4_5.0x5.0mm_P3.2mm, F.Cu at (141.9, 101.0)
- added D5: SK6812, LED_SMD:LED_SK6812_PLCC4_5.0x5.0mm_P3.2mm, F.Cu at (149.9, 80.0)
- added D6: SK6812, LED_SMD:LED_SK6812_PLCC4_5.0x5.0mm_P3.2mm, F.Cu at (149.9, 87.0)
- added D7: SK6812, LED_SMD:LED_SK6812_PLCC4_5.0x5.0mm_P3.2mm, F.Cu at (149.9, 94.0)
- added D8: SK6812, LED_SMD:LED_SK6812_PLCC4_5.0x5.0mm_P3.2mm, F.Cu at (149.9, 101.0)
- added D9: SK6812, LED_SMD:LED_SK6812_PLCC4_5.0x5.0mm_P3.2mm, F.Cu at (157.9, 80.0)
- added H5: MountingHole_Pad, MountingHole:MountingHole_2.2mm_M2_Pad, F.Cu at (162.8, 73.0)
- added H6: MountingHole_Pad, MountingHole:MountingHole_2.2mm_M2_Pad, F.Cu at (162.8, 108.1)
- added H7: MountingHole_Pad, MountingHole:MountingHole_2.2mm_M2_Pad, F.Cu at (137.0, 108.1)
- added H8: MountingHole_Pad, MountingHole:MountingHole_2.2mm_M2_Pad, F.Cu at (137.0, 73.0)
- added J4: Light Bar Connector (main), Connector_PinHeader_2.54mm:PinHeader_1x03_P2.54mm_Vertical, F.Cu at (88.9, 77.3)
- added J5: Light Bar Connector (daughter), Connector_PinSocket_2.54mm:PinSocket_1x03_P2.54mm_Vertical, F.Cu at (136.3, 77.3)
- added R10: 33, Resistor_SMD:R_0402_1005Metric, F.Cu at (139.0, 83.2)
- moved J2 3.00 mm to (110.5, 97.3)
- moved J3 3.00 mm to (90.7, 93.1)
- moved R1 1.46 mm to (99.0, 81.8)
- moved J1 1.22 mm to (102.5, 72.4)
- moved R9 1.16 mm to (91.6, 83.7)
- moved R3 0.64 mm to (91.3, 82.3), turned to -90 degrees
Connections:
- U1 pad 3: unconnected-(U1-GPIO1-Pad3) -> Light bar Signal
Routing:
- net Daughter 5V: track 0.00 -> 112.4 mm, vias 0 -> 6
- net VBUS: track 35.6 -> 65.9 mm
- net Light bar Signal: track 0.00 -> 24.0 mm, vias 0 -> 1
- net Net-(D8-DOUT): track 0.00 -> 21.3 mm, vias 0 -> 2
- net Net-(D4-DOUT): track 0.00 -> 21.2 mm, vias 0 -> 2
- net Net-(D11-DOUT): track 0.00 -> 12.2 mm
- net Net-(D3-DOUT): track 0.00 -> 12.2 mm
- net Net-(D10-DOUT): track 0.00 -> 12.2 mm
- net Net-(D10-DIN): track 0.00 -> 12.2 mm
- net Net-(D7-DOUT): track 0.00 -> 12.2 mm
- net Net-(D6-DOUT): track 0.00 -> 12.2 mm
- net Net-(D5-DOUT): track 0.00 -> 12.2 mm
- net Net-(D2-DOUT): track 0.00 -> 12.2 mm
- net Net-(D1-DOUT): track 0.00 -> 12.2 mm
- net Net-(J5-Pin_2): track 0.00 -> 4.26 mm
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- added copper zone on B.Cu, net Daughter 5V
- added copper zone on F.Cu, net Daughter Ground
Other:
- board size 31.2 x 40.5 mm -> 78.7 x 40.5 mm

Commit message: case
Parts:
- moved H5 15.0 mm to (177.8, 73.0)
- moved H6 15.0 mm to (177.8, 108.1)
- moved C17 14.9 mm to (158.9, 83.5)
- moved C18 14.9 mm to (158.9, 90.5)
- moved C19 14.9 mm to (158.9, 97.5)
- moved C20 14.9 mm to (158.9, 104.5)
- moved C21 14.9 mm to (166.9, 83.5)
- moved C22 14.9 mm to (166.9, 90.5)
- moved C23 14.9 mm to (166.9, 97.5)
- moved C24 14.9 mm to (166.9, 104.5)
- moved C25 14.9 mm to (174.9, 83.5)
- moved C26 14.9 mm to (174.9, 90.5)
- moved C27 14.9 mm to (174.9, 97.5)
- moved C28 14.9 mm to (174.9, 104.5)
- moved C29 14.9 mm to (153.9, 76.8)
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Routing:
- net Light bar Signal: track 24.0 -> 22.8 mm
- net VBUS: track 65.9 -> 64.9 mm, vias 1 -> 0
- net NeoPixel Signal: track 7.02 -> 6.05 mm
- net /PWM Signal: track 4.29 -> 3.68 mm
Other:
- board size 78.7 x 40.5 mm -> 93.6 x 40.5 mm

Commit message: stuff
Parts:
- J2: footprint Connector_PinHeader_2.54mm:PinHeader_1x03_P2.54mm_Horizontal -> Connector_JST:JST_PH_S3B-PH-K_1x03_P2.00mm_Horizontal
- moved J2 4.19 mm to (113.3, 99.1), turned to 90 degrees
- moved J3 2.00 mm to (91.6, 95.1)
- moved C11 1.00 mm to (94.8, 100.1)
- moved C14 1.00 mm to (94.8, 101.0)
Connections:
- J2 pad 1: /PWM GND -> /PWM Signal
- J2 pad 3: /PWM Signal -> /PWM GND
Routing:
- net VBUS: track 64.9 -> 59.9 mm
- net /PWM Signal: track 3.68 -> 8.49 mm
- net /PWM GND: track 12.1 -> 15.9 mm
- net NeoPixel Signal: track 6.05 -> 5.22 mm
- net +3V3: track 20.2 -> 20.9 mm

Commit message: journal
Parts:
- moved C29 7.27 mm to (161.2, 76.3)
- moved J4 2.00 mm to (88.9, 79.3)
- moved J5 2.00 mm to (151.2, 79.3)
- moved U3 1.55 mm to (95.3, 87.1)
Routing:
- net VBUS: track 59.9 -> 47.5 mm
- net Daughter 5V: track 112.4 -> 120.7 mm
- net /RP2040 Circuitry/FLASH_SS: track 20.8 -> 17.9 mm
- net /RP2040 Circuitry/FLASH_0: track 8.06 -> 10.8 mm
- net Light bar Signal: track 22.8 -> 20.8 mm
- net /RP2040 Circuitry/FLASH_1: track 16.4 -> 14.4 mm
- net +3V3: track 20.9 -> 19.0 mm
- net Net-(J5-Pin_2): track 4.26 -> 2.74 mm
- net /RP2040 Circuitry/FLASH_2: track 12.6 -> 11.6 mm
- net /RP2040 Circuitry/FLASH_CLK: track 10.4 -> 11.3 mm, vias 0 -> 2
- net /RP2040 Circuitry/FLASH_3: track 11.5 -> 12.1 mm

Commit message: whoops i forgot to commit this
Parts:
- removed R10: 33, Resistor_SMD:R_0402_1005Metric
- added mouse-bite-2mm-slot: VAL**, jank:mouse-bite-2mm-slot, F.Cu at (119.1, 90.5)
- added mouse-bite-2mm-slot: VAL**, jank:mouse-bite-2mm-slot, F.Cu at (119.1, 75.3)
- added mouse-bite-2mm-slot: VAL**, jank:mouse-bite-2mm-slot, F.Cu at (119.1, 105.8)
- C17, C18, C19, C20, C21, C22, C23, C24, C25, C26, C27, C28: value 0.1u -> 100n
- C29: footprint Capacitor_SMD:C_0402_1005Metric -> Capacitor_SMD:C_1206_3216Metric
- U4: footprint LTV-217-B-G:SOIC127P700X210-4N -> LTV-357T:LTV-357T_LTO
- moved H5 29.2 mm to (148.6, 73.0)
- moved H6 29.2 mm to (148.6, 108.1)
- moved D1 29.2 mm to (127.7, 80.0)
- moved D2 29.2 mm to (127.7, 87.0)
- moved D3 29.2 mm to (127.7, 94.0)
- moved D4 29.2 mm to (127.7, 101.0)
- moved J5 29.2 mm to (122.0, 79.3)
- moved C17 29.2 mm to (129.7, 83.5)
- moved C18 29.2 mm to (129.7, 90.5)
- moved C19 29.2 mm to (129.7, 97.5)
- moved C20 29.2 mm to (129.7, 104.5)
- moved C21 29.2 mm to (137.7, 83.5)
- moved C22 29.2 mm to (137.7, 90.5)
- moved C23 29.2 mm to (137.7, 97.5)
- moved C24 29.2 mm to (137.7, 104.5)
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Connections:
- J5 pad 2: Net-(J5-Pin_2) -> Net-(D1-DIN)
Routing:
- net Daughter 5V: track 120.7 -> 123.6 mm
- net Net-(J5-Pin_2): track 2.74 -> 0.00 mm
- net Net-(D1-DIN): track 1.67 -> 3.32 mm
- net GND: track 37.4 -> 36.2 mm
- net PWM Signal GPIO: track 13.3 -> 14.2 mm
- net /PWM GND: track 15.9 -> 15.2 mm
Other:
- board size 93.6 x 40.5 mm -> 64.4 x 40.5 mm
- board text added: "DEV REV_1"
