File: Hardware/v0/NeoPWM.kicad_sch (KiCad schematic)
At the start: 9 parts, among them J2 PWM Input, J3 NeoPixel Connector, U4 LTV-357T

Commit message: he
Parts:
- added C17, C18, C19, C20, C21, C22, C23, C24, C25, C26, C27, C28: 0.1u, Capacitor_SMD:C_0402_1005Metric, symbol Device:C
- added C29: 100u, Capacitor_SMD:C_0402_1005Metric, symbol Device:C
- added D1, D10, D11, D12, D2, D3, D4, D5, D6, D7, D8, D9: SK6812, LED_SMD:LED_SK6812_PLCC4_5.0x5.0mm_P3.2mm, symbol LED:SK6812
- added H5, H6, H7, H8: MountingHole_Pad, MountingHole:MountingHole_2.2mm_M2_Pad, symbol Mechanical:MountingHole_Pad
- added J4: Light Bar Connector (main), Connector_PinHeader_2.54mm:PinHeader_1x03_P2.54mm_Vertical, symbol Connector:Conn_01x03_Pin
- added J5: Light Bar Connector (daughter), Connector_PinSocket_2.54mm:PinSocket_1x03_P2.54mm_Vertical, symbol Connector:Conn_01x03_Socket
- added R10: 33, Resistor_SMD:R_0402_1005Metric, symbol Device:R
Connections:
- net GND: now also J4.3 (Pin_3)
- net VBUS: now also J4.1 (Pin_1)
- new net: D11.4 (DOUT), D12.2 (DIN)
- new net: D8.4 (DOUT), D9.2 (DIN)
- new net: D10.2 (DIN), D9.4 (DOUT)
- new net: D1.4 (DOUT), D2.2 (DIN)
- new net: D2.4 (DOUT), D3.2 (DIN)
- new net: D5.4 (DOUT), D6.2 (DIN)
- new net: D6.4 (DOUT), D7.2 (DIN)
- new net: D3.4 (DOUT), D4.2 (DIN)
- new net: D7.4 (DOUT), D8.2 (DIN)
- new net: D4.4 (DOUT), D5.2 (DIN)
- new net: D1.2 (DIN), R10.2
- new net: D10.4 (DOUT), D11.2 (DIN)
- new net: J5.2 (Pin_2), R10.1
- new net Daughter 5V: C17.1, C18.1, C19.1, C20.1, C21.1, C22.1, C23.1, C24.1, C25.1, C26.1, C27.1, C28.1, C29.1, D1.3 (VDD), D10.3 (VDD), D11.3 (VDD), D12.3 (VDD), D2.3 (VDD), D3.3 (VDD), D4.3 (VDD), D5.3 (VDD), D6.3 (VDD), D7.3 (VDD), D8.3 (VDD), D9.3 (VDD), J5.1 (Pin_1)
- new net Daughter Ground: C17.2, C18.2, C19.2, C20.2, C21.2, C22.2, C23.2, C24.2, C25.2, C26.2, C27.2, C28.2, C29.2, D1.1 (VSS), D10.1 (VSS), D11.1 (VSS), D12.1 (VSS), D2.1 (VSS), D3.1 (VSS), D4.1 (VSS), D5.1 (VSS), D6.1 (VSS), D7.1 (VSS), D8.1 (VSS), D9.1 (VSS), H5.1, H6.1, H7.1, H8.1, J5.3 (Pin_3)
- new net Light bar Signal: J4.2 (Pin_2)
Other:
- note added: "Daughter board"

Commit message: stuff
Parts:
- J2: footprint Connector_PinHeader_2.54mm:PinHeader_1x03_P2.54mm_Horizontal -> Connector_JST:JST_PH_S3B-PH-K_1x03_P2.00mm_Horizontal
Connections:
- net PWM GND: now also J2.3 (Pin_3); no longer J2.1 (Pin_1)
- net PWM Signal: now also J2.1 (Pin_1); no longer J2.3 (Pin_3)
Changed lines of the file:
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@@
+	(wire
+		(pts
+			(xy 132.08 39.37) (xy 127 39.37)
+		)
+		(stroke
+			(width 0)
+			(type default)
+		)
+	)
 	(wire
 		(pts
@@
 	(wire
 		(pts
-			(xy 127 39.37) (xy 132.08 39.37)
-		)
-		(stroke
-			(width 0)
-			(type default)
-		)
-	)
-	(wire
-		(pts
 			(xy 134.62 120.65) (xy 144.78 120.65)
 		)
@@
 	(wire
 		(pts
+			(xy 114.3 152.4) (xy 104.14 152.4)
+		)
+		(stroke
+			(width 0)
+			(type default)
+		)
+	)
+	(wire
+		(pts
+			(xy 111.76 137.16) (xy 116.84 137.16)
+		)
+		(stroke
+			(width 0)
+			(type default)
+		)
+	)
+	(wire
+		(pts
+			(xy 58.42 160.02) (xy 76.2 160.02)
+		)
+		(stroke
+			(width 0)
+			(type default)
+		)
+	)
+	(wire
+		(pts
+			(xy 93.98 116.84) (xy 93.98 120.65)
+		)
+		(stroke
+			(width 0)
+			(type default)
+		)
+	)
+	(wire
+		(pts
+			(xy 167.64 162.56) (xy 190.5 162.56)
+		)
+		(stroke
+			(width 0)
+			(type default)
+		)
+	)
+	(wire
+		(pts
+			(xy 172.72 113.03) (xy 176.53 113.03)
+		)
+		(stroke
+			(width 0)
+			(type default)
+		)
+	)
+	(wire
+		(pts
+			(xy 114.3 156.21) (xy 114.3 152.4)
+		)
+		(stroke
+			(width 0)
+			(type default)
+		)
+	)
+	(wire
+		(pts
+			(xy 154.94 120.65) (xy 165.1 120.65)
+		)
+		(stroke
+			(width 0)
+			(type default)
+		)
+	)
+	(wire
+		(pts
+			(xy 132.08 113.03) (xy 137.16 113.03)
+		)
+		(stroke
+			(width 0)
+			(type default)
+		)
+	)
+	(wire
+		(pts
+			(xy 114.3 129.54) (xy 114.3 133.35)
+		)
+		(stroke
+			(width 0)
+			(type default)
+		)
+	)
+	(wire
+		(pts
+			(xy 83.82 152.4) (xy 93.98 152.4)
+		)
+		(stroke
+			(width 0)
+			(type default)
+		)
+	)
+	(wire
+		(pts
+			(xy 154.94 129.54) (xy 154.94 133.35)
+		)
+		(stroke
+			(width 0)
+			(type default)
+		)
+	)
+	(wire
+		(pts
+			(xy 154.94 144.78) (xy 165.1 144.78)
+		)
+		(stroke
+			(width 0)
+			(type default)
+		)
+	)
+	(wire
+		(pts
+			(xy 124.46 144.78) (xy 134.62 144.78)
+		)
+		(stroke
+			(width 0)
+			(type default)
+		)
+	)
+	(wire
+		(pts
+			(xy 114.3 144.78) (xy 124.46 144.78)
+		)
+		(stroke
+			(width 0)
+			(type default)
+		)
+	)
+	(wire
+		(pts
 			(xy 127 44.45) (xy 132.08 44.45)
-		)
-		(stroke
-			(width 0)
-			(type default)
-		)
-	)
-	(wire
-		(pts
-			(xy 114.3 152.4) (xy 104.14 152.4)
-		)
-		(stroke
-			(width 0)
-			(type default)
-		)
-	)
-	(wire
-		(pts
-			(xy 111.76 137.16) (xy 116.84 137.16)
-		)
-		(stroke
-			(width 0)
-			(type default)
-		)
-	)
-	(wire
-		(pts
-			(xy 58.42 160.02) (xy 76.2 160.02)
-		)
-		(stroke
-			(width 0)
-			(type default)
-		)
-	)
-	(wire
-		(pts
-			(xy 93.98 116.84) (xy 93.98 120.65)
-		)
-		(stroke
-			(width 0)
-			(type default)
-		)
-	)
-	(wire
-		(pts
-			(xy 167.64 162.56) (xy 190.5 162.56)
-		)
-		(stroke
-			(width 0)
-			(type default)
-		)
-	)
-	(wire
-		(pts
-			(xy 172.72 113.03) (xy 176.53 113.03)
-		)
-		(stroke
-			(width 0)
-			(type default)
-		)
-	)
-	(wire
-		(pts
-			(xy 114.3 156.21) (xy 114.3 152.4)
-		)
-		(stroke
-			(width 0)
-			(type default)
-		)
-	)
-	(wire
-		(pts
-			(xy 154.94 120.65) (xy 165.1 120.65)
-		)
-		(stroke
-			(width 0)
-			(type default)
-		)
-	)
-	(wire
-		(pts
-			(xy 132.08 113.03) (xy 137.16 113.03)
-		)
-		(stroke
-			(width 0)
-			(type default)
-		)
-	)
-	(wire
-		(pts
-			(xy 114.3 129.54) (xy 114.3 133.35)
-		)
-		(stroke
-			(width 0)
-			(type default)
-		)
-	)
-	(wire
-		(pts
-			(xy 83.82 152.4) (xy 93.98 152.4)
-		)
-		(stroke
-			(width 0)
-			(type default)
-		)
-	)
-	(wire
-		(pts
-			(xy 154.94 129.54) (xy 154.94 133.35)
-		)
-		(stroke
-			(width 0)
-			(type default)
-		)
-	)
-	(wire
-		(pts
-			(xy 154.94 144.78) (xy 165.1 144.78)
-		)
-		(stroke
-			(width 0)
-			(type default)
-		)
-	)
-	(wire
-		(pts
-			(xy 124.46 144.78) (xy 134.62 144.78)
-		)
-		(stroke
-			(width 0)
-			(type default)
-		)
-	)
-	(wire
-		(pts
-			(xy 114.3 144.78) (xy 124.46 144.78)
 		)
 		(stroke
@@
 	)
 	(label "PWM GND"
-		(at 132.08 39.37 0)
+		(at 132.08 44.45 0)
 		(effects
 			(font
@@
 	)
 	(label "PWM Signal"
-		(at 132.08 44.45 0)
+		(at 132.08 39.37 0)
 		(effects
 			(font
@@
 			)
 		)
-		(property "Footprint" "Connector_PinHeader_2.54mm:PinHeader_1x03_P2.54mm_Horizontal"
+		(property "Footprint" "Connector_JST:JST_PH_S3B-PH-K_1x03_P2.00mm_Horizontal"
 			(at 121.92 41.91 0)
 			(effects

Commit message: whoops i forgot to commit this
Parts:
- removed R10: 33, Resistor_SMD:R_0402_1005Metric, symbol Device:R
- C17, C18, C19, C20, C21, C22, C23, C24, C25, C26, C27, C28: value 0.1u -> 100n; LCSC (none) -> C1525
- C29: footprint Capacitor_SMD:C_0402_1005Metric -> Capacitor_SMD:C_1206_3216Metric; LCSC (none) -> C15008
- D1, D10, D11, D12, D2, D3, D4, D5, D6, D7, D8, D9: LCSC (none) -> C5380878
- J2, J3, J4, J5: now left out of the parts list
- R5: LCSC (none) -> C25117
- R6: LCSC (none) -> C25900
- U4: footprint LTV-217-B-G:SOIC127P700X210-4N -> LTV-357T:LTV-357T_LTO; LCSC (none) -> C119089
Connections:
- net at D1.2 (DIN): now also J5.2 (Pin_2)
